File: kicad/binary_clock/binary_clock.kicad_pcb (KiCad board)
At the start: 2 copper layers, 74 x 84 mm, 39 parts, among them J1 USB_B_Micro, J2 ISP, J3 DCF-77 Receiver, SW1 SLEEP, U3 ATmega328P-PU

Commit message: Added Quarz Oscillator.
Parts:
- added C4: 22pF, Capacitor_SMD:C_0805_2012Metric_Pad1.15x1.40mm_HandSolder, B.Cu at (108.6, 124.5)
- added C5: 22pF, Capacitor_SMD:C_0805_2012Metric_Pad1.15x1.40mm_HandSolder, B.Cu at (113.5, 124.5)
- added Y1: 16MHz, Crystal:Crystal_HC49-U_Vertical, B.Cu at (113.5, 119.0)
- moved C1 40.5 mm to (148.0, 110.5), turned to 90 degrees
Connections:
- U3 pad 10: Net-(R12-Pad1) -> /XTAL2
- U3 pad 5: Net-(U3-Pad5) -> Net-(R11-Pad1)
- U3 pad 6: Net-(U3-Pad6) -> Net-(R12-Pad1)
- U3 pad 9: Net-(R11-Pad1) -> /XTAL1
Routing:
- net /XTAL2: track 0.00 -> 12.1 mm
- net /XTAL1: track 0.00 -> 10.8 mm
- net +5V: track 86.9 -> 95.9 mm, vias 1 -> 2
- net Net-(R12-Pad1): track 34.1 -> 39.6 mm
- net Net-(R11-Pad1): track 22.7 -> 27.8 mm
